File: LCD_Breakout/LCD_breakout.brd (EAGLE design)
At the start: 32.9 x 63.7 mm, 12 parts

Commit message: Add files via upload
Parts:
- removed JP4: (no value), pinhead:1X02
- R3: device rcl:R1206 -> rcl:0204/5
- moved R3 4.83 mm to (17.4, 6.85)
- moved R1 3.00 mm to (7.62, 56.3)
- moved JP1 2.00 mm to (7.62, 24.9)
- moved JP2 2.00 mm to (16.6, 19.8)
- moved JP3 2.00 mm to (16.6, 33.8)
- moved JP5 2.00 mm to (16.6, 42.6)
- moved LED1 2.00 mm to (23.4, 54.5)
- moved R2 2.00 mm to (17.5, 54.5)
- moved SV1 2.00 mm to (27.0, 39.0)
- moved SV2 2.00 mm to (27.0, 17.0)
- moved U$1 2.00 mm to (-8.00, 11.9)
Connections:
- removed net N$17: JP4.1, R3.2
- removed net N$19: JP1.1, JP4.2, U$1.16
- net +5V: now also R3.2
- net GND: now also JP1.1, U$1.16
Routing:
- net +5V: track 135.4 -> 122.6 mm
- net N$19: track 9.67 -> 0.00 mm
- net N$18: track 3.64 -> 7.93 mm
- net N$17: track 2.61 -> 0.00 mm
- net GND: track 9.60 -> 10.9 mm
- net N$1: track 22.4 -> 23.4 mm
