File: Atmega16_32/Atmega32_Dev.brd (EAGLE design)
At the start: 105 x 65 mm, 35 parts, among them IC1 MEGA32-P, J1 DCJ0202

Commit message: Add files via upload
Parts:
- added JP2, JP3: (no value), pinhead:1X05
- added LED9: (no value), led:LED3MM
- added R10: 1k, rcl:0204/7
- C1, C2: value (none) -> 22pF
- C3, C4: value (none) -> 100uF
- C5: value (none) -> 100nF
- L1: value (none) -> 100uH
- Q1: value (none) -> 12MHz
- R1, R2, R3, R4, R5, R6, R7, R8: value (none) -> 1k
- R9: value (none) -> 10k
- flipped R9 to the top
Connections:
- new net N$9: LED9.A, R10.1
- net +5V: now also JP2.1, JP2.2, JP2.3, JP2.4, JP2.5, R10.2
- net GND: now also JP3.1, JP3.2, JP3.3, JP3.4, JP3.5, LED9.K
Routing:
- net +5V: track 351.2 -> 375.5 mm
- net RESET: track 151.1 -> 145.5 mm
- net N$9: track 0.00 -> 5.22 mm
- net GND: track 125.6 -> 124.1 mm
Other:
- board text added: "+5V"
- board text added: "0"
- board text added: "12MHz"
- board text added: "ARef"
- board text added: "AVcc"
- board text added: "GND"

Commit message: Add files via upload
Parts:
- removed JP2, JP3: (no value), pinhead:1X05
- removed LED9: (no value), led:LED3MM
- removed R10: 1k, rcl:0204/7
- C1, C2: value 22pF -> (none)
- C3, C4: value 100uF -> (none)
- C5: value 100nF -> (none)
- L1: value 100uH -> (none)
- Q1: value 12MHz -> (none)
- R1, R2, R3, R4, R5, R6, R7, R8: value 1k -> (none)
- R9: value 10k -> (none)
- flipped R9 to the bottom
Connections:
- removed net N$9: LED9.A, R10.1
- net +5V: no longer JP2.1, JP2.2, JP2.3, JP2.4, JP2.5, R10.2
- net GND: no longer JP3.1, JP3.2, JP3.3, JP3.4, JP3.5, LED9.K
- net PB5: now also ISP.9; no longer ISP.1
- net PB6: now also ISP.1; no longer ISP.9
Routing:
- net GND: track 124.1 -> 157.7 mm
- net +5V: track 375.5 -> 351.6 mm
- net PB6: track 56.9 -> 44.4 mm
- net PB5: track 58.9 -> 49.2 mm
- net RESET: track 145.5 -> 148.8 mm
- net N$10: track 0.00 -> 3.25 mm
- net N$11: track 0.00 -> 2.35 mm
- net N$9: track 5.22 -> 3.10 mm
Other:
- board text removed: "+5V"
- board text removed: "0"
- board text removed: "12MHz"
- board text removed: "ARef"
- board text removed: "AVcc"
- board text removed: "GND"
