File: Atmega16_32/Atmega32_Dev.sch (EAGLE design)
At the start: 35 parts, among them IC1 MEGA32-P, J1 DCJ0202

Commit message: Add files via upload
Parts:
- added JP2, JP3: (no value), pinhead:PINHD-1X5
- added LED9: (no value), led:LED3MM
- added R10: 1k, rcl:R-EU_0204/7
- C1, C2: value (none) -> 22pF
- C3, C4: value (none) -> 100uF
- C5: value (none) -> 100nF
- L1: value (none) -> 100uH
- Q1: value (none) -> 12MHz
- R1, R2, R3, R4, R5, R6, R7, R8: value (none) -> 1k
- R9: value (none) -> 10k
Connections:
- new net N$9: LED9.A, R10.1
- net +5V: now also JP2.1, JP2.2, JP2.3, JP2.4, JP2.5, R10.2
- net GND: now also JP3.1, JP3.2, JP3.3, JP3.4, JP3.5, LED9.C
Changed lines of the file:
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@@
 <part name="LED7" library="led" deviceset="LED" device="3MM"/>
 <part name="LED8" library="led" deviceset="LED" device="3MM"/>
-<part name="R1" library="resistor" deviceset="R-EU_" device="M1206"/>
-<part name="R2" library="resistor" deviceset="R-EU_" device="M1206"/>
-<part name="R3" library="resistor" deviceset="R-EU_" device="M1206"/>
-<part name="R4" library="resistor" deviceset="R-EU_" device="M1206"/>
-<part name="R5" library="resistor" deviceset="R-EU_" device="M1206"/>
-<part name="R6" library="resistor" deviceset="R-EU_" device="M1206"/>
-<part name="R7" library="resistor" deviceset="R-EU_" device="M1206"/>
-<part name="R8" library="resistor" deviceset="R-EU_" device="M1206"/>
+<part name="R1" library="resistor" deviceset="R-EU_" device="M1206" value="1k"/>
+<part name="R2" library="resistor" deviceset="R-EU_" device="M1206" value="1k"/>
+<part name="R3" library="resistor" deviceset="R-EU_" device="M1206" value="1k"/>
+<part name="R4" library="resistor" deviceset="R-EU_" device="M1206" value="1k"/>
+<part name="R5" library="resistor" deviceset="R-EU_" device="M1206" value="1k"/>
+<part name="R6" library="resistor" deviceset="R-EU_" device="M1206" value="1k"/>
+<part name="R7" library="resistor" deviceset="R-EU_" device="M1206" value="1k"/>
+<part name="R8" library="resistor" deviceset="R-EU_" device="M1206" value="1k"/>
 <part name="GND1" library="supply1" deviceset="GND" device=""/>
 <part name="P+1" library="supply1" deviceset="+5V" device=""/>
@@
 <part name="P+2" library="supply1" deviceset="+12V" device=""/>
 <part name="IC2" library="v-reg" deviceset="78XXL" device=""/>
-<part name="L1" library="rcl" deviceset="L-US" device="0204/5"/>
+<part name="L1" library="rcl" deviceset="L-US" device="0204/5" value="100uH"/>
 <part name="P+3" library="supply1" deviceset="+5V" device=""/>
 <part name="GND3" library="supply1" deviceset="GND" device=""/>
 <part name="S1" library="switch-omron" deviceset="10-XX" device=""/>
 <part name="GND4" library="supply1" deviceset="GND" device=""/>
-<part name="R9" library="rcl" deviceset="R-EU_" device="0204/7"/>
+<part name="R9" library="rcl" deviceset="R-EU_" device="0204/7" value="10k"/>
 <part name="P+4" library="supply1" deviceset="+5V" device=""/>
-<part name="C1" library="SparkFun" deviceset="CAP" device="1206"/>
-<part name="C2" library="SparkFun" deviceset="CAP" device="1206"/>
+<part name="C1" library="SparkFun" deviceset="CAP" device="1206" value="22pF"/>
+<part name="C2" library="SparkFun" deviceset="CAP" device="1206" value="22pF"/>
 <part name="GND5" library="supply1" deviceset="GND" device=""/>
-<part name="C3" library="rcl" deviceset="CPOL-EU" device="E5-6"/>
-<part name="C4" library="rcl" deviceset="CPOL-EU" device="E5-6"/>
-<part name="C5" library="SparkFun" deviceset="CAP" device="1206"/>
+<part name="C3" library="rcl" deviceset="CPOL-EU" device="E5-6" value="100uF"/>
+<part name="C4" library="rcl" deviceset="CPOL-EU" device="E5-6" value="100uF"/>
+<part name="C5" library="SparkFun" deviceset="CAP" device="1206" value="100nF"/>
 <part name="J1" library="con-jack" deviceset="DCJ0202" device=""/>
-<part name="Q1" library="SmartPrj" deviceset="XTAL/S" device=""/>
+<part name="Q1" library="SmartPrj" deviceset="XTAL/S" device="" value="12MHz"/>
 <part name="JP1" library="pinhead" deviceset="PINHD-1X2" device=""/>
+<part name="JP2" library="pinhead" deviceset="PINHD-1X5" device=""/>
+<part name="JP3" library="pinhead" deviceset="PINHD-1X5" device=""/>
+<part name="P+5" library="supply1" deviceset="+5V" device=""/>
+<part name="GND6" library="supply1" deviceset="GND" device=""/>
+<part name="LED9" library="led" deviceset="LED" device="3MM"/>
+<part name="R10" library="rcl" deviceset="R-EU_" device="0204/7" value="1k"/>
+<part name="GND7" library="supply1" deviceset="GND" device=""/>
+<part name="P+6" library="supply1" deviceset="+5V" device=""/>
 </parts>
 <sheets>
@@
 <instance part="Q1" gate="G$1" x="63.5" y="119.38"/>
 <instance part="JP1" gate="G$1" x="129.54" y="160.02" rot="R180"/>
+<instance part="JP2" gate="A" x="175.26" y="152.4" rot="R180"/>
+<instance part="JP3" gate="A" x="157.48" y="152.4" rot="R180"/>
+<instance part="P+5" gate="1" x="187.96" y="162.56"/>
+<instance part="GND6" gate="1" x="167.64" y="139.7"/>
+<instance part="LED9" gate="G$1" x="114.3" y="160.02"/>
+<instance part="R10" gate="G$1" x="114.3" y="167.64" rot="R90"/>
+<instance part="GND7" gate="1" x="114.3" y="152.4"/>
+<instance part="P+6" gate="1" x="114.3" y="175.26"/>
 </instances>
 <busses>
@@
 <wire x1="152.4" y1="96.52" x2="149.86" y2="96.52" width="0.1524" layer="91"/>
 </segment>
+<segment>
+<pinref part="JP3" gate="A" pin="5"/>
+<pinref part="GND6" gate="1" pin="GND"/>
+<wire x1="160.02" y1="157.48" x2="167.64" y2="157.48" width="0.1524" layer="91"/>
+<wire x1="167.64" y1="157.48" x2="167.64" y2="154.94" width="0.1524" layer="91"/>
+<pinref part="JP3" gate="A" pin="2"/>
+<wire x1="167.64" y1="154.94" x2="167.64" y2="152.4" width="0.1524" layer="91"/>
+<wire x1="167.64" y1="152.4" x2="167.64" y2="149.86" width="0.1524" layer="91"/>
+<wire x1="167.64" y1="149.86" x2="167.64" y2="147.32" width="0.1524" layer="91"/>
+<wire x1="167.64" y1="147.32" x2="167.64" y2="142.24" width="0.1524" layer="91"/>
+<wire x1="160.02" y1="149.86" x2="167.64" y2="149.86" width="0.1524" layer="91"/>
+<pinref part="JP3" gate="A" pin="4"/>
+<wire x1="160.02" y1="154.94" x2="167.64" y2="154.94" width="0.1524" layer="91"/>
+<pinref part="JP3" gate="A" pin="3"/>
+<wire x1="160.02" y1="152.4" x2="167.64" y2="152.4" width="0.1524" layer="91"/>
+<pinref part="JP3" gate="A" pin="1"/>
+<wire x1="160.02" y1="147.32" x2="167.64" y2="147.32" width="0.1524" layer="91"/>
+<junction x="167.64" y="154.94"/>
+<junction x="167.64" y="152.4"/>
+<junction x="167.64" y="149.86"/>
+<junction x="167.64" y="147.32"/>
+</segment>
+<segment>
+<pinref part="GND7" gate="1" pin="GND"/>
+<pinref part="LED9" gate="G$1" pin="C"/>
+</segment>
 </net>
 <net name="PA7" class="0">
@@
 <pinref part="ISP" gate="G$1" pin="2"/>
 <wire x1="152.4" y1="88.9" x2="149.86" y2="88.9" width="0.1524" layer="91"/>
+</segment>
+<segment>
+<pinref part="JP2" gate="A" pin="1"/>
+<pinref part="P+5" gate="1" pin="+5V"/>
+<wire x1="177.8" y1="147.32" x2="187.96" y2="147.32" width="0.1524" layer="91"/>
+<wire x1="187.96" y1="147.32" x2="187.96" y2="149.86" width="0.1524" layer="91"/>
+<pinref part="JP2" gate="A" pin="2"/>
+<wire x1="187.96" y1="149.86" x2="187.96" y2="152.4" width="0.1524" layer="91"/>
+<wire x1="187.96" y1="154.94" x2="187.96" y2="157.48" width="0.1524" layer="91"/>
+<wire x1="187.96" y1="157.48" x2="187.96" y2="160.02" width="0.1524" layer="91"/>
+<wire x1="177.8" y1="149.86" x2="187.96" y2="149.86" width="0.1524" layer="91"/>
+<pinref part="JP2" gate="A" pin="3"/>
+<wire x1="177.8" y1="152.4" x2="187.96" y2="152.4" width="0.1524" layer="91"/>
+<wire x1="187.96" y1="152.4" x2="187.96" y2="154.94" width="0.1524" layer="91"/>
+<pinref part="JP2" gate="A" pin="4"/>
+<wire x1="177.8" y1="154.94" x2="187.96" y2="154.94" width="0.1524" layer="91"/>
+<pinref part="JP2" gate="A" pin="5"/>
+<wire x1="177.8" y1="157.48" x2="187.96" y2="157.48" width="0.1524" layer="91"/>
+<junction x="187.96" y="149.86"/>
+<junction x="187.96" y="152.4"/>
+<junction x="187.96" y="154.94"/>
+<junction x="187.96" y="157.48"/>
+</segment>
+<segment>
+<pinref part="P+6" gate="1" pin="+5V"/>
+<pinref part="R10" gate="G$1" pin="2"/>
 </segment>
 </net>
@@
 </segment>
 </net>
+<net name="N$9" class="0">
+<segment>
+<pinref part="R10" gate="G$1" pin="1"/>
+<pinref part="LED9" gate="G$1" pin="A"/>
+</segment>
+</net>

Commit message: Add files via upload
Parts:
- removed JP2, JP3: (no value), pinhead:PINHD-1X5
- removed LED9: (no value), led:LED3MM
- removed R10: 1k, rcl:R-EU_0204/7
- C1, C2: value 22pF -> (none)
- C3, C4: value 100uF -> (none)
- C5: value 100nF -> (none)
- L1: value 100uH -> (none)
- Q1: value 12MHz -> (none)
- R1, R2, R3, R4, R5, R6, R7, R8: value 1k -> (none)
- R9: value 10k -> (none)
Connections:
- removed net N$9: LED9.A, R10.1
- net +5V: no longer JP2.1, JP2.2, JP2.3, JP2.4, JP2.5, R10.2
- net GND: no longer JP3.1, JP3.2, JP3.3, JP3.4, JP3.5, LED9.C
- net PB5: now also ISP.9; no longer ISP.1
- net PB6: now also ISP.1; no longer ISP.9
Changed lines of the file:
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@@
 <part name="LED7" library="led" deviceset="LED" device="3MM"/>
 <part name="LED8" library="led" deviceset="LED" device="3MM"/>
-<part name="R1" library="resistor" deviceset="R-EU_" device="M1206" value="1k"/>
-<part name="R2" library="resistor" deviceset="R-EU_" device="M1206" value="1k"/>
-<part name="R3" library="resistor" deviceset="R-EU_" device="M1206" value="1k"/>
-<part name="R4" library="resistor" deviceset="R-EU_" device="M1206" value="1k"/>
-<part name="R5" library="resistor" deviceset="R-EU_" device="M1206" value="1k"/>
-<part name="R6" library="resistor" deviceset="R-EU_" device="M1206" value="1k"/>
-<part name="R7" library="resistor" deviceset="R-EU_" device="M1206" value="1k"/>
-<part name="R8" library="resistor" deviceset="R-EU_" device="M1206" value="1k"/>
+<part name="R1" library="resistor" deviceset="R-EU_" device="M1206"/>
+<part name="R2" library="resistor" deviceset="R-EU_" device="M1206"/>
+<part name="R3" library="resistor" deviceset="R-EU_" device="M1206"/>
+<part name="R4" library="resistor" deviceset="R-EU_" device="M1206"/>
+<part name="R5" library="resistor" deviceset="R-EU_" device="M1206"/>
+<part name="R6" library="resistor" deviceset="R-EU_" device="M1206"/>
+<part name="R7" library="resistor" deviceset="R-EU_" device="M1206"/>
+<part name="R8" library="resistor" deviceset="R-EU_" device="M1206"/>
 <part name="GND1" library="supply1" deviceset="GND" device=""/>
 <part name="P+1" library="supply1" deviceset="+5V" device=""/>
@@
 <part name="P+2" library="supply1" deviceset="+12V" device=""/>
 <part name="IC2" library="v-reg" deviceset="78XXL" device=""/>
-<part name="L1" library="rcl" deviceset="L-US" device="0204/5" value="100uH"/>
+<part name="L1" library="rcl" deviceset="L-US" device="0204/5"/>
 <part name="P+3" library="supply1" deviceset="+5V" device=""/>
 <part name="GND3" library="supply1" deviceset="GND" device=""/>
 <part name="S1" library="switch-omron" deviceset="10-XX" device=""/>
 <part name="GND4" library="supply1" deviceset="GND" device=""/>
-<part name="R9" library="rcl" deviceset="R-EU_" device="0204/7" value="10k"/>
+<part name="R9" library="rcl" deviceset="R-EU_" device="0204/7"/>
 <part name="P+4" library="supply1" deviceset="+5V" device=""/>
-<part name="C1" library="SparkFun" deviceset="CAP" device="1206" value="22pF"/>
-<part name="C2" library="SparkFun" deviceset="CAP" device="1206" value="22pF"/>
+<part name="C1" library="SparkFun" deviceset="CAP" device="1206"/>
+<part name="C2" library="SparkFun" deviceset="CAP" device="1206"/>
 <part name="GND5" library="supply1" deviceset="GND" device=""/>
-<part name="C3" library="rcl" deviceset="CPOL-EU" device="E5-6" value="100uF"/>
-<part name="C4" library="rcl" deviceset="CPOL-EU" device="E5-6" value="100uF"/>
-<part name="C5" library="SparkFun" deviceset="CAP" device="1206" value="100nF"/>
+<part name="C3" library="rcl" deviceset="CPOL-EU" device="E5-6"/>
+<part name="C4" library="rcl" deviceset="CPOL-EU" device="E5-6"/>
+<part name="C5" library="SparkFun" deviceset="CAP" device="1206"/>
 <part name="J1" library="con-jack" deviceset="DCJ0202" device=""/>
-<part name="Q1" library="SmartPrj" deviceset="XTAL/S" device="" value="12MHz"/>
+<part name="Q1" library="SmartPrj" deviceset="XTAL/S" device=""/>
 <part name="JP1" library="pinhead" deviceset="PINHD-1X2" device=""/>
-<part name="JP2" library="pinhead" deviceset="PINHD-1X5" device=""/>
-<part name="JP3" library="pinhead" deviceset="PINHD-1X5" device=""/>
-<part name="P+5" library="supply1" deviceset="+5V" device=""/>
-<part name="GND6" library="supply1" deviceset="GND" device=""/>
-<part name="LED9" library="led" deviceset="LED" device="3MM"/>
-<part name="R10" library="rcl" deviceset="R-EU_" device="0204/7" value="1k"/>
-<part name="GND7" library="supply1" deviceset="GND" device=""/>
-<part name="P+6" library="supply1" deviceset="+5V" device=""/>
 </parts>
 <sheets>
@@
 <instance part="Q1" gate="G$1" x="63.5" y="119.38"/>
 <instance part="JP1" gate="G$1" x="129.54" y="160.02" rot="R180"/>
-<instance part="JP2" gate="A" x="175.26" y="152.4" rot="R180"/>
-<instance part="JP3" gate="A" x="157.48" y="152.4" rot="R180"/>
-<instance part="P+5" gate="1" x="187.96" y="162.56"/>
-<instance part="GND6" gate="1" x="167.64" y="139.7"/>
-<instance part="LED9" gate="G$1" x="114.3" y="160.02"/>
-<instance part="R10" gate="G$1" x="114.3" y="167.64" rot="R90"/>
-<instance part="GND7" gate="1" x="114.3" y="152.4"/>
-<instance part="P+6" gate="1" x="114.3" y="175.26"/>
 </instances>
 <busses>
@@
 <wire x1="152.4" y1="96.52" x2="149.86" y2="96.52" width="0.1524" layer="91"/>
 </segment>
-<segment>
-<pinref part="JP3" gate="A" pin="5"/>
-<pinref part="GND6" gate="1" pin="GND"/>
-<wire x1="160.02" y1="157.48" x2="167.64" y2="157.48" width="0.1524" layer="91"/>
-<wire x1="167.64" y1="157.48" x2="167.64" y2="154.94" width="0.1524" layer="91"/>
-<pinref part="JP3" gate="A" pin="2"/>
-<wire x1="167.64" y1="154.94" x2="167.64" y2="152.4" width="0.1524" layer="91"/>
-<wire x1="167.64" y1="152.4" x2="167.64" y2="149.86" width="0.1524" layer="91"/>
-<wire x1="167.64" y1="149.86" x2="167.64" y2="147.32" width="0.1524" layer="91"/>
-<wire x1="167.64" y1="147.32" x2="167.64" y2="142.24" width="0.1524" layer="91"/>
-<wire x1="160.02" y1="149.86" x2="167.64" y2="149.86" width="0.1524" layer="91"/>
-<pinref part="JP3" gate="A" pin="4"/>
-<wire x1="160.02" y1="154.94" x2="167.64" y2="154.94" width="0.1524" layer="91"/>
-<pinref part="JP3" gate="A" pin="3"/>
-<wire x1="160.02" y1="152.4" x2="167.64" y2="152.4" width="0.1524" layer="91"/>
-<pinref part="JP3" gate="A" pin="1"/>
-<wire x1="160.02" y1="147.32" x2="167.64" y2="147.32" width="0.1524" layer="91"/>
-<junction x="167.64" y="154.94"/>
-<junction x="167.64" y="152.4"/>
-<junction x="167.64" y="149.86"/>
-<junction x="167.64" y="147.32"/>
-</segment>
-<segment>
-<pinref part="GND7" gate="1" pin="GND"/>
-<pinref part="LED9" gate="G$1" pin="C"/>
-</segment>
 </net>
 <net name="PA7" class="0">
@@
 <wire x1="152.4" y1="88.9" x2="149.86" y2="88.9" width="0.1524" layer="91"/>
 </segment>
-<segment>
-<pinref part="JP2" gate="A" pin="1"/>
-<pinref part="P+5" gate="1" pin="+5V"/>
-<wire x1="177.8" y1="147.32" x2="187.96" y2="147.32" width="0.1524" layer="91"/>
-<wire x1="187.96" y1="147.32" x2="187.96" y2="149.86" width="0.1524" layer="91"/>
-<pinref part="JP2" gate="A" pin="2"/>
-<wire x1="187.96" y1="149.86" x2="187.96" y2="152.4" width="0.1524" layer="91"/>
-<wire x1="187.96" y1="154.94" x2="187.96" y2="157.48" width="0.1524" layer="91"/>
-<wire x1="187.96" y1="157.48" x2="187.96" y2="160.02" width="0.1524" layer="91"/>
-<wire x1="177.8" y1="149.86" x2="187.96" y2="149.86" width="0.1524" layer="91"/>
-<pinref part="JP2" gate="A" pin="3"/>
-<wire x1="177.8" y1="152.4" x2="187.96" y2="152.4" width="0.1524" layer="91"/>
-<wire x1="187.96" y1="152.4" x2="187.96" y2="154.94" width="0.1524" layer="91"/>
-<pinref part="JP2" gate="A" pin="4"/>
-<wire x1="177.8" y1="154.94" x2="187.96" y2="154.94" width="0.1524" layer="91"/>
-<pinref part="JP2" gate="A" pin="5"/>
-<wire x1="177.8" y1="157.48" x2="187.96" y2="157.48" width="0.1524" layer="91"/>
-<junction x="187.96" y="149.86"/>
-<junction x="187.96" y="152.4"/>
-<junction x="187.96" y="154.94"/>
-<junction x="187.96" y="157.48"/>
-</segment>
-<segment>
-<pinref part="P+6" gate="1" pin="+5V"/>
-<pinref part="R10" gate="G$1" pin="2"/>
-</segment>
 </net>
 <net name="N$44" class="0">
@@
 </segment>
 <segment>
+<pinref part="ISP" gate="G$1" pin="1"/>
+<wire x1="167.64" y1="88.9" x2="170.18" y2="88.9" width="0.1524" layer="91"/>
+</segment>
+</net>
+<net name="PB7" class="0">
+<segment>
+<pinref part="PORTB" gate="G$1" pin="8"/>
+<wire x1="27.94" y1="96.52" x2="25.4" y2="96.52" width="0.1524" layer="91"/>
+</segment>
+<segment>
+<pinref part="IC1" gate="G$1" pin="(SCK)PB7"/>
+<wire x1="119.38" y1="111.76" x2="121.92" y2="111.76" width="0.1524" layer="91"/>
+</segment>
+<segment>
+<pinref part="ISP" gate="G$1" pin="7"/>
+<wire x1="167.64" y1="96.52" x2="170.18" y2="96.52" width="0.1524" layer="91"/>
+</segment>
+</net>
+<net name="PB5" class="0">
+<segment>
+<pinref part="PORTB" gate="G$1" pin="6"/>
+<wire x1="27.94" y1="93.98" x2="25.4" y2="93.98" width="0.1524" layer="91"/>
+</segment>
+<segment>
+<pinref part="IC1" gate="G$1" pin="(MOSI)PB5"/>
+<wire x1="119.38" y1="106.68" x2="121.92" y2="106.68" width="0.1524" layer="91"/>
+</segment>
+<segment>
 <pinref part="ISP" gate="G$1" pin="9"/>
 <wire x1="167.64" y1="99.06" x2="170.18" y2="99.06" width="0.1524" layer="91"/>
-</segment>
-</net>
-<net name="PB7" class="0">
-<segment>
-<pinref part="PORTB" gate="G$1" pin="8"/>
-<wire x1="27.94" y1="96.52" x2="25.4" y2="96.52" width="0.1524" layer="91"/>
-</segment>
-<segment>
-<pinref part="IC1" gate="G$1" pin="(SCK)PB7"/>
-<wire x1="119.38" y1="111.76" x2="121.92" y2="111.76" width="0.1524" layer="91"/>
-</segment>
-<segment>
-<pinref part="ISP" gate="G$1" pin="7"/>
-<wire x1="167.64" y1="96.52" x2="170.18" y2="96.52" width="0.1524" layer="91"/>
-</segment>
-</net>
-<net name="PB5" class="0">
-<segment>
-<pinref part="PORTB" gate="G$1" pin="6"/>
-<wire x1="27.94" y1="93.98" x2="25.4" y2="93.98" width="0.1524" layer="91"/>
-</segment>
-<segment>
-<pinref part="IC1" gate="G$1" pin="(MOSI)PB5"/>
-<wire x1="119.38" y1="106.68" x2="121.92" y2="106.68" width="0.1524" layer="91"/>
-</segment>
-<segment>
-<pinref part="ISP" gate="G$1" pin="1"/>
-<wire x1="167.64" y1="88.9" x2="170.18" y2="88.9" width="0.1524" layer="91"/>
 </segment>
 </net>
@@
 </segment>
 </net>
-<net name="N$9" class="0">
-<segment>
-<pinref part="R10" gate="G$1" pin="1"/>
-<pinref part="LED9" gate="G$1" pin="A"/>
-</segment>
-</net>
