File: Programmer/USBasp_A.brd (EAGLE design)
At the start: 25.8 x 67.9 mm, 20 parts, among them IC1 ATMega8, Q1 12MHz

Commit message: Add files via upload
Parts:
- moved LED2 1.04 mm to (20.7, 36.6)
- moved R4 0.84 mm to (20.9, 31.5)
Connections:
- removed net N$3: IC1.18, X2.1
- new net N$26: IC1.18, X2.9
- net N$6: now also X2.1; no longer X2.9
Routing:
- net N$3: track 60.3 -> 0.00 mm
- net N$26: track 0.00 -> 39.7 mm
- net N$6: track 41.4 -> 53.3 mm
- net +5V: track 128.4 -> 129.6 mm
- net N$13: track 2.26 -> 3.36 mm
Changed lines of the file:
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@@
 <element name="C1" library="rcl" package="E2,5-5" value="4u7" x="22.18" y="13.03" smashed="yes"/>
 <element name="R6" library="rcl" package="R1206W" value="10k" x="5.28" y="50.97" smashed="yes" rot="MR90"/>
-<element name="LED2" library="led" package="LED3MM" value="red" x="20.76" y="35.57" smashed="yes" rot="R90">
-<attribute name="VALUE" x="23.911" y="34.875" size="0.8128" layer="21" ratio="10" rot="R90"/>
+<element name="LED2" library="led" package="LED3MM" value="red" x="20.74" y="36.61" smashed="yes" rot="R90">
+<attribute name="VALUE" x="23.891" y="35.915" size="0.8128" layer="21" ratio="10" rot="R90"/>
 </element>
-<element name="R4" library="rcl" package="R1206W" value="1k" x="21.09" y="30.68" smashed="yes" rot="MR90"/>
+<element name="R4" library="rcl" package="R1206W" value="1k" x="20.94" y="31.51" smashed="yes" rot="MR90"/>
 <element name="JP2" library="jumper" package="JP1" value="Self programming" x="6.52" y="55.4" smashed="yes" rot="R270"/>
 <element name="JP4" library="jumper" package="JP1" value="Clk&gt;1.5MHz" x="20.2" y="48.84" smashed="yes">
@@
 <wire x1="20.6" y1="52.079" x2="21.801" y2="52.079" width="0.4064" layer="16"/>
 <wire x1="21.801" y1="52.079" x2="21.801" y2="52.039" width="0.4064" layer="16"/>
-<wire x1="16.88" y1="32.35" x2="18.09" y2="32.35" width="0.4064" layer="16"/>
-<wire x1="18.09" y1="32.35" x2="20.1" y2="30.34" width="0.4064" layer="16"/>
 <wire x1="22.599" y1="40.28" x2="22.86" y2="40.28" width="0.4064" layer="16"/>
 <wire x1="22.86" y1="40.28" x2="22.9" y2="40.24" width="0.4064" layer="16"/>
 <wire x1="22.9" y1="30.991" x2="21.4345" y2="29.5255" width="0.4064" layer="16"/>
-<wire x1="21.4345" y1="29.5255" x2="21.09" y2="29.181" width="0.4064" layer="16"/>
-<wire x1="21.09" y1="29.181" x2="20.91" y2="29.181" width="0.4064" layer="16"/>
+<wire x1="21.4345" y1="29.5255" x2="20.94" y2="30.011" width="0.4064" layer="16"/>
+<wire x1="20.94" y1="30.011" x2="20.91" y2="29.181" width="0.4064" layer="16"/>
 <wire x1="20.91" y1="29.181" x2="20.91" y2="13.03" width="0.4064" layer="16"/>
-<wire x1="20.1" y1="30.34" x2="20.1" y2="30.32" width="0.4064" layer="16"/>
-<wire x1="20.1" y1="30.32" x2="20.18" y2="30.24" width="0.4064" layer="16"/>
-<wire x1="20.18" y1="30.24" x2="20.72" y2="30.24" width="0.4064" layer="16"/>
 <wire x1="20.72" y1="30.24" x2="21.4345" y2="29.5255" width="0.4064" layer="16"/>
 <wire x1="6.4" y1="37.43" x2="6.4" y2="48.351" width="0.4064" layer="16"/>
@@
 <wire x1="12.43" y1="12.04" x2="15.51" y2="12.04" width="0.4064" layer="16"/>
 <wire x1="15.51" y1="12.04" x2="15.69" y2="12.22" width="0.4064" layer="16"/>
+<wire x1="16.88" y1="32.35" x2="18.601" y2="32.35" width="0.4064" layer="16"/>
+<wire x1="18.601" y1="32.35" x2="20.94" y2="30.011" width="0.4064" layer="16"/>
 </signal>
 <signal name="N$7">
@@
 <contactref element="IC1" pad="16"/>
 <contactref element="JP2" pad="2"/>
-<wire x1="12.9" y1="60.41" x2="12.9" y2="24.04" width="0.4064" layer="16"/>
+<wire x1="12.9" y1="60.41" x2="12.9" y2="24.04" width="0.3048" layer="16"/>
 <wire x1="12.9" y1="24.04" x2="14.9" y2="22.04" width="0.4064" layer="16"/>
 <wire x1="14.9" y1="22.04" x2="16.73" y2="22.04" width="0.4064" layer="16"/>
 <wire x1="16.73" y1="22.04" x2="16.88" y2="22.19" width="0.4064" layer="16"/>
-<wire x1="12.9" y1="60.41" x2="12.63" y2="60.41" width="0.3048" layer="16"/>
-<wire x1="12.63" y1="60.41" x2="11.2" y2="61.84" width="0.3048" layer="16"/>
-<wire x1="11.2" y1="61.84" x2="7.2" y2="61.84" width="0.3048" layer="16"/>
-<wire x1="7.2" y1="61.84" x2="6.4" y2="61.04" width="0.3048" layer="16"/>
-<wire x1="6.4" y1="61.04" x2="6.4" y2="58.84" width="0.3048" layer="16"/>
-<wire x1="6.4" y1="58.84" x2="7.7" y2="57.54" width="0.3048" layer="16"/>
-<wire x1="7.7" y1="57.54" x2="7.7" y2="55.49" width="0.3048" layer="16"/>
-<wire x1="7.7" y1="55.49" x2="7.79" y2="55.4" width="0.3048" layer="16"/>
+<wire x1="7.79" y1="55.4" x2="7.79" y2="57.69" width="0.4064" layer="16"/>
+<wire x1="7.79" y1="57.69" x2="6.26" y2="59.22" width="0.4064" layer="16"/>
+<wire x1="6.26" y1="59.22" x2="6.26" y2="60.91" width="0.4064" layer="16"/>
+<wire x1="6.26" y1="60.91" x2="7" y2="61.65" width="0.4064" layer="16"/>
+<wire x1="7" y1="61.65" x2="12.2" y2="61.65" width="0.4064" layer="16"/>
+<wire x1="12.2" y1="61.65" x2="12.9" y2="60.95" width="0.4064" layer="16"/>
+<wire x1="12.9" y1="60.95" x2="12.9" y2="60.41" width="0.4064" layer="16"/>
 </signal>
 <signal name="N$4">
@@
 <contactref element="LED2" pad="A"/>
 <contactref element="R4" pad="2"/>
-<wire x1="20.76" y1="34.3" x2="20.76" y2="32.509" width="0.4064" layer="16"/>
-<wire x1="20.76" y1="32.509" x2="21.09" y2="32.179" width="0.4064" layer="16"/>
+<wire x1="20.74" y1="35.34" x2="20.76" y2="32.509" width="0.4064" layer="16"/>
+<wire x1="20.76" y1="32.509" x2="20.94" y2="33.009" width="0.4064" layer="16"/>
 </signal>
 <signal name="N$14">
 <contactref element="IC1" pad="23"/>
 <contactref element="LED2" pad="K"/>
-<wire x1="17.07" y1="39.97" x2="20.1" y2="36.94" width="0.4064" layer="16"/>
-<wire x1="20.1" y1="36.94" x2="20.66" y2="36.94" width="0.4064" layer="16"/>
-<wire x1="20.66" y1="36.94" x2="20.76" y2="36.84" width="0.4064" layer="16"/>
 <wire x1="16.88" y1="39.97" x2="17.07" y2="39.97" width="0.4064" layer="16"/>
+<wire x1="17.07" y1="39.97" x2="17.07" y2="39.74" width="0.4064" layer="16"/>
+<wire x1="17.07" y1="39.74" x2="18.92" y2="37.89" width="0.4064" layer="16"/>
+<wire x1="18.92" y1="37.89" x2="20.73" y2="37.89" width="0.4064" layer="16"/>
+<wire x1="20.73" y1="37.89" x2="20.74" y2="37.88" width="0.4064" layer="16"/>
 </signal>
 <signal name="N$15">
@@
 <wire x1="4.78" y1="16.559" x2="4.571" y2="16.35" width="0.4064" layer="16"/>
 </signal>
-<signal name="N$3">
+<signal name="N$6">
+<contactref element="IC1" pad="17"/>
 <contactref element="X2" pad="1"/>
-<contactref element="IC1" pad="18"/>
-<wire x1="16.88" y1="27.27" x2="15.23" y2="27.27" width="0.3048" layer="16"/>
-<wire x1="15.23" y1="27.27" x2="13.9" y2="25.94" width="0.3048" layer="16"/>
-<wire x1="13.9" y1="25.94" x2="13.9" y2="24.14" width="0.3048" layer="16"/>
-<wire x1="13.9" y1="24.14" x2="14.6" y2="23.47" width="0.3048" layer="16"/>
-<wire x1="14.6" y1="23.47" x2="18.9" y2="23.47" width="0.3048" layer="16"/>
-<wire x1="18.9" y1="23.47" x2="19.5" y2="22.84" width="0.3048" layer="16"/>
-<wire x1="19.5" y1="22.84" x2="19.5" y2="21.44" width="0.3048" layer="16"/>
-<wire x1="7.82" y1="60.41" x2="7.82" y2="58.52" width="0.4064" layer="16"/>
-<wire x1="7.82" y1="58.52" x2="12.1" y2="54.24" width="0.4064" layer="16"/>
-<wire x1="12.1" y1="54.24" x2="12.1" y2="23.44" width="0.4064" layer="16"/>
-<wire x1="12.1" y1="23.44" x2="14.64" y2="20.92" width="0.4064" layer="16"/>
-<wire x1="14.64" y1="20.92" x2="18.98" y2="20.92" width="0.3048" layer="16"/>
-<wire x1="18.98" y1="20.92" x2="19.5" y2="21.44" width="0.3048" layer="16"/>
-</signal>
-<signal name="N$6">
-<contactref element="X2" pad="9"/>
-<contactref element="IC1" pad="17"/>
-<wire x1="18.15" y1="31.08" x2="19.42" y2="29.81" width="0.3048" layer="16"/>
-<wire x1="19.42" y1="29.81" x2="19.42" y2="27.27" width="0.3048" layer="16"/>
-<wire x1="19.42" y1="27.27" x2="16.88" y2="24.73" width="0.3048" layer="16"/>
-<wire x1="14.9" y1="53.84" x2="14.9" y2="31.74" width="0.4064" layer="16"/>
-<wire x1="14.9" y1="53.84" x2="16.8" y2="55.74" width="0.4064" layer="16"/>
-<wire x1="16.8" y1="55.74" x2="16.8" y2="59.23" width="0.4064" layer="16"/>
-<wire x1="16.8" y1="59.23" x2="17.98" y2="60.41" width="0.4064" layer="16"/>
-<wire x1="18.15" y1="31.08" x2="15.56" y2="31.08" width="0.3048" layer="16"/>
-<wire x1="15.56" y1="31.08" x2="14.9" y2="31.74" width="0.3048" layer="16"/>
+<wire x1="16.88" y1="24.73" x2="18.15" y2="24.73" width="0.4064" layer="16"/>
+<wire x1="18.15" y1="24.73" x2="18.92" y2="23.96" width="0.4064" layer="16"/>
+<wire x1="18.92" y1="23.96" x2="18.92" y2="21.67" width="0.4064" layer="16"/>
+<wire x1="18.92" y1="21.67" x2="18.2" y2="20.95" width="0.4064" layer="16"/>
+<wire x1="18.2" y1="20.95" x2="14.36" y2="20.95" width="0.4064" layer="16"/>
+<wire x1="14.36" y1="20.95" x2="12" y2="23.31" width="0.4064" layer="16"/>
+<wire x1="12" y1="23.31" x2="12" y2="57.8" width="0.3048" layer="16"/>
+<wire x1="12" y1="57.8" x2="11.07" y2="58.73" width="0.4064" layer="16"/>
+<wire x1="11.07" y1="58.73" x2="8.37" y2="58.73" width="0.4064" layer="16"/>
+<wire x1="8.37" y1="58.73" x2="7.75" y2="59.35" width="0.4064" layer="16"/>
+<wire x1="7.75" y1="59.35" x2="7.75" y2="60.34" width="0.4064" layer="16"/>
+<wire x1="7.75" y1="60.34" x2="7.82" y2="60.41" width="0.4064" layer="16"/>
 </signal>
 <signal name="N$9">
@@
 <wire x1="17.68" y1="45.05" x2="20.2" y2="47.57" width="0.4064" layer="16"/>
 </signal>
+<signal name="N$26">
+<contactref element="IC1" pad="18"/>
+<contactref element="X2" pad="9"/>
+<wire x1="17.98" y1="60.41" x2="17.98" y2="56.75" width="0.4064" layer="16"/>
+<wire x1="17.98" y1="56.75" x2="14.85" y2="53.62" width="0.4064" layer="16"/>
+<wire x1="14.85" y1="53.62" x2="14.85" y2="31.56" width="0.4064" layer="16"/>
+<wire x1="14.85" y1="31.56" x2="15.32" y2="31.09" width="0.4064" layer="16"/>
+<wire x1="15.32" y1="31.09" x2="18.08" y2="31.09" width="0.4064" layer="16"/>
+<wire x1="18.08" y1="31.09" x2="19.29" y2="29.88" width="0.4064" layer="16"/>
+<wire x1="19.29" y1="29.88" x2="19.29" y2="28.37" width="0.4064" layer="16"/>
+<wire x1="19.29" y1="28.37" x2="18.23" y2="27.31" width="0.4064" layer="16"/>
+<wire x1="18.23" y1="27.31" x2="16.92" y2="27.31" width="0.4064" layer="16"/>
+<wire x1="16.92" y1="27.31" x2="16.88" y2="27.27" width="0.4064" layer="16"/>
+</signal>
 </signals>

Commit message: Add files via upload
Connections:
- removed net N$6: IC1.17, X2.1
- new net N$3: IC1.17, X2.9
- net N$26: now also X2.1; no longer X2.9
Routing:
- net N$6: track 53.3 -> 0.00 mm
- net N$3: track 0.00 -> 47.2 mm
- net N$26: track 39.7 -> 55.4 mm
Changed lines of the file:
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@@
 </polygon>
 <contactref element="JP4" pad="2"/>
-<wire x1="16.88" y1="37.43" x2="9.26" y2="34.89" width="0" layer="19" extent="1-1"/>
+<wire x1="9.26" y1="34.89" x2="16.88" y2="37.43" width="0" layer="19" extent="1-1"/>
 </signal>
 <signal name="N$5">
@@
 <wire x1="7.79" y1="55.4" x2="7.79" y2="57.69" width="0.4064" layer="16"/>
 <wire x1="7.79" y1="57.69" x2="6.26" y2="59.22" width="0.4064" layer="16"/>
-<wire x1="6.26" y1="59.22" x2="6.26" y2="60.91" width="0.4064" layer="16"/>
-<wire x1="6.26" y1="60.91" x2="7" y2="61.65" width="0.4064" layer="16"/>
-<wire x1="7" y1="61.65" x2="12.2" y2="61.65" width="0.4064" layer="16"/>
-<wire x1="12.2" y1="61.65" x2="12.9" y2="60.95" width="0.4064" layer="16"/>
-<wire x1="12.9" y1="60.95" x2="12.9" y2="60.41" width="0.4064" layer="16"/>
+<wire x1="6.26" y1="59.22" x2="6.3" y2="60.9" width="0.4064" layer="16"/>
+<wire x1="6.3" y1="60.9" x2="7.04" y2="61.67" width="0.4064" layer="16"/>
+<wire x1="7.04" y1="61.67" x2="12.17" y2="61.68" width="0.4064" layer="16"/>
+<wire x1="12.17" y1="61.68" x2="12.87" y2="60.95" width="0.4064" layer="16"/>
+<wire x1="12.87" y1="60.95" x2="12.9" y2="60.41" width="0.4064" layer="16"/>
 </signal>
 <signal name="N$4">
@@
 <wire x1="4.78" y1="16.559" x2="4.571" y2="16.35" width="0.4064" layer="16"/>
 </signal>
-<signal name="N$6">
-<contactref element="IC1" pad="17"/>
-<contactref element="X2" pad="1"/>
-<wire x1="16.88" y1="24.73" x2="18.15" y2="24.73" width="0.4064" layer="16"/>
-<wire x1="18.15" y1="24.73" x2="18.92" y2="23.96" width="0.4064" layer="16"/>
-<wire x1="18.92" y1="23.96" x2="18.92" y2="21.67" width="0.4064" layer="16"/>
-<wire x1="18.92" y1="21.67" x2="18.2" y2="20.95" width="0.4064" layer="16"/>
-<wire x1="18.2" y1="20.95" x2="14.36" y2="20.95" width="0.4064" layer="16"/>
-<wire x1="14.36" y1="20.95" x2="12" y2="23.31" width="0.4064" layer="16"/>
-<wire x1="12" y1="23.31" x2="12" y2="57.8" width="0.3048" layer="16"/>
-<wire x1="12" y1="57.8" x2="11.07" y2="58.73" width="0.4064" layer="16"/>
-<wire x1="11.07" y1="58.73" x2="8.37" y2="58.73" width="0.4064" layer="16"/>
-<wire x1="8.37" y1="58.73" x2="7.75" y2="59.35" width="0.4064" layer="16"/>
-<wire x1="7.75" y1="59.35" x2="7.75" y2="60.34" width="0.4064" layer="16"/>
-<wire x1="7.75" y1="60.34" x2="7.82" y2="60.41" width="0.4064" layer="16"/>
-</signal>
 <signal name="N$9">
 </signal>
@@
 <signal name="N$26">
 <contactref element="IC1" pad="18"/>
+<contactref element="X2" pad="1"/>
+<wire x1="16.88" y1="27.27" x2="18.11" y2="27.27" width="0.4064" layer="16"/>
+<wire x1="18.11" y1="27.27" x2="19.41" y2="25.97" width="0.4064" layer="16"/>
+<wire x1="19.41" y1="25.97" x2="19.41" y2="22" width="0.4064" layer="16"/>
+<wire x1="19.41" y1="22" x2="18.42" y2="21.01" width="0.4064" layer="16"/>
+<wire x1="18.42" y1="21.01" x2="18.42" y2="20.98" width="0.4064" layer="16"/>
+<wire x1="18.42" y1="20.98" x2="18.36" y2="20.92" width="0.4064" layer="16"/>
+<wire x1="18.36" y1="20.92" x2="14.49" y2="20.92" width="0.4064" layer="16"/>
+<wire x1="14.49" y1="20.92" x2="12.13" y2="23.28" width="0.4064" layer="16"/>
+<wire x1="12.13" y1="23.28" x2="12.13" y2="23.3" width="0.4064" layer="16"/>
+<wire x1="12.13" y1="23.3" x2="12.06" y2="23.37" width="0.4064" layer="16"/>
+<wire x1="12.06" y1="23.37" x2="12.06" y2="57.47" width="0.3048" layer="16"/>
+<wire x1="12.06" y1="57.47" x2="11.01" y2="58.52" width="0.4064" layer="16"/>
+<wire x1="11.01" y1="58.52" x2="9.71" y2="58.52" width="0.4064" layer="16"/>
+<wire x1="9.71" y1="58.52" x2="7.82" y2="60.41" width="0.4064" layer="16"/>
+</signal>
+<signal name="N$3">
 <contactref element="X2" pad="9"/>
-<wire x1="17.98" y1="60.41" x2="17.98" y2="56.75" width="0.4064" layer="16"/>
-<wire x1="17.98" y1="56.75" x2="14.85" y2="53.62" width="0.4064" layer="16"/>
-<wire x1="14.85" y1="53.62" x2="14.85" y2="31.56" width="0.4064" layer="16"/>
-<wire x1="14.85" y1="31.56" x2="15.32" y2="31.09" width="0.4064" layer="16"/>
-<wire x1="15.32" y1="31.09" x2="18.08" y2="31.09" width="0.4064" layer="16"/>
-<wire x1="18.08" y1="31.09" x2="19.29" y2="29.88" width="0.4064" layer="16"/>
-<wire x1="19.29" y1="29.88" x2="19.29" y2="28.37" width="0.4064" layer="16"/>
-<wire x1="19.29" y1="28.37" x2="18.23" y2="27.31" width="0.4064" layer="16"/>
-<wire x1="18.23" y1="27.31" x2="16.92" y2="27.31" width="0.4064" layer="16"/>
-<wire x1="16.92" y1="27.31" x2="16.88" y2="27.27" width="0.4064" layer="16"/>
+<contactref element="IC1" pad="17"/>
+<wire x1="17.98" y1="60.41" x2="17.98" y2="56.62" width="0.4064" layer="16"/>
+<wire x1="17.98" y1="56.62" x2="14.92" y2="53.56" width="0.4064" layer="16"/>
+<wire x1="16.88" y1="24.73" x2="15.04" y2="24.73" width="0.4064" layer="16"/>
+<wire x1="15.04" y1="24.73" x2="13.86" y2="25.91" width="0.4064" layer="16"/>
+<wire x1="13.86" y1="25.91" x2="13.86" y2="27.7" width="0.4064" layer="16"/>
+<wire x1="13.86" y1="27.7" x2="14.67" y2="28.51" width="0.4064" layer="16"/>
+<wire x1="14.67" y1="28.51" x2="18.45" y2="28.51" width="0.4064" layer="16"/>
+<wire x1="18.45" y1="28.51" x2="19.01" y2="29.07" width="0.4064" layer="16"/>
+<wire x1="19.01" y1="29.07" x2="19.01" y2="30.62" width="0.4064" layer="16"/>
+<wire x1="19.01" y1="30.62" x2="18.54" y2="31.09" width="0.4064" layer="16"/>
+<wire x1="18.54" y1="31.09" x2="15.26" y2="31.09" width="0.4064" layer="16"/>
+<wire x1="15.26" y1="31.09" x2="14.92" y2="31.43" width="0.4064" layer="16"/>
+<wire x1="14.92" y1="31.43" x2="14.92" y2="53.56" width="0.4064" layer="16"/>
 </signal>
 </signals>
