File: Programmer/USBasp_B.brd (EAGLE design)
At the start: 25.7 x 64.6 mm, 20 parts, among them IC1 ATMega8, Q1 12MHz

Commit message: Add files via upload
Parts:
- moved LED2 0.58 mm to (21.2, 32.8)
- moved R4 0.51 mm to (21.3, 27.8)
Connections:
- removed net N$6: IC1.17, X2.9
- new net N$27: IC1.18, X2.9
- net N$3: now also IC1.17; no longer IC1.18
Routing:
- net N$6: track 41.4 -> 0.00 mm
- net N$27: track 0.00 -> 39.5 mm
- net N$3: track 60.3 -> 53.1 mm
- net N$2: track 54.9 -> 55.5 mm
Changed lines of the file:
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@@
 <element name="C1" library="rcl" package="E2,5-5" value="4u7" x="22.58" y="9.69" smashed="yes"/>
 <element name="R6" library="rcl" package="R1206W" value="10k" x="5.68" y="47.63" smashed="yes" rot="MR90"/>
-<element name="LED2" library="led" package="LED3MM" value="red" x="21.16" y="32.23" smashed="yes" rot="R90">
-<attribute name="VALUE" x="24.311" y="31.535" size="0.8128" layer="21" ratio="10" rot="R90"/>
+<element name="LED2" library="led" package="LED3MM" value="red" x="21.16" y="32.81" smashed="yes" rot="R90">
+<attribute name="VALUE" x="24.311" y="32.115" size="0.8128" layer="21" ratio="10" rot="R90"/>
 </element>
-<element name="R4" library="rcl" package="R1206W" value="1k" x="21.49" y="27.34" smashed="yes" rot="MR90"/>
+<element name="R4" library="rcl" package="R1206W" value="1k" x="21.28" y="27.81" smashed="yes" rot="MR90"/>
 <element name="JP2" library="jumper" package="JP1" value="Self programming" x="6.92" y="52.06" smashed="yes" rot="R270"/>
 <element name="JP4" library="jumper" package="JP1" value="Clk&gt;1.5MHz" x="20.6" y="45.5" smashed="yes">
@@
 </polygon>
 <contactref element="JP4" pad="2"/>
-<wire x1="17.28" y1="34.09" x2="9.66" y2="31.55" width="0" layer="19" extent="1-1"/>
+<wire x1="9.66" y1="31.55" x2="17.28" y2="34.09" width="0" layer="19" extent="1-1"/>
 </signal>
 <signal name="N$5">
@@
 <wire x1="21" y1="48.739" x2="22.201" y2="48.739" width="0.4064" layer="16"/>
 <wire x1="22.201" y1="48.739" x2="22.201" y2="48.699" width="0.4064" layer="16"/>
-<wire x1="17.28" y1="29.01" x2="18.49" y2="29.01" width="0.4064" layer="16"/>
-<wire x1="18.49" y1="29.01" x2="20.5" y2="27" width="0.4064" layer="16"/>
 <wire x1="22.999" y1="36.94" x2="23.26" y2="36.94" width="0.4064" layer="16"/>
 <wire x1="23.26" y1="36.94" x2="23.3" y2="36.9" width="0.4064" layer="16"/>
-<wire x1="23.3" y1="27.651" x2="21.8345" y2="26.1855" width="0.4064" layer="16"/>
-<wire x1="21.8345" y1="26.1855" x2="21.49" y2="25.841" width="0.4064" layer="16"/>
-<wire x1="21.49" y1="25.841" x2="21.31" y2="25.841" width="0.4064" layer="16"/>
+<wire x1="23.3" y1="27.651" x2="21.28" y2="26.311" width="0.4064" layer="16"/>
+<wire x1="21.28" y1="26.311" x2="21.31" y2="25.841" width="0.4064" layer="16"/>
 <wire x1="21.31" y1="25.841" x2="21.31" y2="9.69" width="0.4064" layer="16"/>
-<wire x1="20.5" y1="27" x2="20.5" y2="26.98" width="0.4064" layer="16"/>
-<wire x1="20.5" y1="26.98" x2="20.58" y2="26.9" width="0.4064" layer="16"/>
-<wire x1="20.58" y1="26.9" x2="21.12" y2="26.9" width="0.4064" layer="16"/>
-<wire x1="21.12" y1="26.9" x2="21.8345" y2="26.1855" width="0.4064" layer="16"/>
 <wire x1="20.31" y1="8.69" x2="21.31" y2="9.69" width="0.4064" layer="16"/>
 <wire x1="14.429" y1="8.341" x2="14.45" y2="8.32" width="0.4064" layer="16"/>
@@
 <wire x1="6.8" y1="34.09" x2="6.8" y2="45.011" width="0.4064" layer="16"/>
 <wire x1="6.8" y1="45.011" x2="5.68" y2="46.131" width="0.4064" layer="16"/>
+<wire x1="17.28" y1="29.01" x2="18.581" y2="29.01" width="0.4064" layer="16"/>
+<wire x1="18.581" y1="29.01" x2="21.28" y2="26.311" width="0.4064" layer="16"/>
 </signal>
 <signal name="N$7">
@@
 <wire x1="15.3" y1="18.7" x2="17.13" y2="18.7" width="0.4064" layer="16"/>
 <wire x1="17.13" y1="18.7" x2="17.28" y2="18.85" width="0.4064" layer="16"/>
-<wire x1="13.3" y1="57.07" x2="13.03" y2="57.07" width="0.3048" layer="16"/>
-<wire x1="13.03" y1="57.07" x2="11.6" y2="58.5" width="0.3048" layer="16"/>
-<wire x1="11.6" y1="58.5" x2="7.6" y2="58.5" width="0.3048" layer="16"/>
-<wire x1="7.6" y1="58.5" x2="6.8" y2="57.7" width="0.3048" layer="16"/>
-<wire x1="6.8" y1="57.7" x2="6.8" y2="55.5" width="0.3048" layer="16"/>
 <wire x1="6.8" y1="55.5" x2="8.1" y2="54.2" width="0.3048" layer="16"/>
 <wire x1="8.1" y1="54.2" x2="8.1" y2="52.15" width="0.3048" layer="16"/>
 <wire x1="8.1" y1="52.15" x2="8.19" y2="52.06" width="0.3048" layer="16"/>
+<wire x1="13.3" y1="57.07" x2="13.3" y2="57.21" width="0.4064" layer="16"/>
+<wire x1="13.3" y1="57.21" x2="12.2" y2="58.31" width="0.3048" layer="16"/>
+<wire x1="12.2" y1="58.31" x2="6.91" y2="58.31" width="0.3048" layer="16"/>
+<wire x1="6.91" y1="58.31" x2="6.33" y2="57.73" width="0.3048" layer="16"/>
+<wire x1="6.33" y1="57.73" x2="6.33" y2="55.97" width="0.3048" layer="16"/>
+<wire x1="6.33" y1="55.97" x2="6.8" y2="55.5" width="0.3048" layer="16"/>
 </signal>
 <signal name="N$4">
@@
 <contactref element="LED2" pad="A"/>
 <contactref element="R4" pad="2"/>
-<wire x1="21.16" y1="30.96" x2="21.16" y2="29.169" width="0.4064" layer="16"/>
-<wire x1="21.16" y1="29.169" x2="21.49" y2="28.839" width="0.4064" layer="16"/>
+<wire x1="21.16" y1="31.54" x2="21.16" y2="29.169" width="0.4064" layer="16"/>
+<wire x1="21.16" y1="29.169" x2="21.28" y2="29.309" width="0.4064" layer="16"/>
 </signal>
 <signal name="N$14">
 <contactref element="IC1" pad="23"/>
 <contactref element="LED2" pad="K"/>
-<wire x1="17.47" y1="36.63" x2="20.5" y2="33.6" width="0.4064" layer="16"/>
-<wire x1="20.5" y1="33.6" x2="21.06" y2="33.6" width="0.4064" layer="16"/>
-<wire x1="21.06" y1="33.6" x2="21.16" y2="33.5" width="0.4064" layer="16"/>
 <wire x1="17.28" y1="36.63" x2="17.47" y2="36.63" width="0.4064" layer="16"/>
+<wire x1="17.47" y1="36.63" x2="17.47" y2="36.55" width="0.4064" layer="16"/>
+<wire x1="17.47" y1="36.55" x2="19.98" y2="34.04" width="0.4064" layer="16"/>
+<wire x1="19.98" y1="34.04" x2="21.12" y2="34.04" width="0.4064" layer="16"/>
+<wire x1="21.12" y1="34.04" x2="21.16" y2="34.08" width="0.4064" layer="16"/>
 </signal>
 <signal name="N$15">
@@
 <signal name="N$3">
 <contactref element="X2" pad="1"/>
-<contactref element="IC1" pad="18"/>
-<wire x1="17.28" y1="23.93" x2="15.63" y2="23.93" width="0.3048" layer="16"/>
-<wire x1="15.63" y1="23.93" x2="14.3" y2="22.6" width="0.3048" layer="16"/>
-<wire x1="14.3" y1="22.6" x2="14.3" y2="20.8" width="0.3048" layer="16"/>
-<wire x1="14.3" y1="20.8" x2="15" y2="20.13" width="0.3048" layer="16"/>
-<wire x1="15" y1="20.13" x2="19.3" y2="20.13" width="0.3048" layer="16"/>
-<wire x1="19.3" y1="20.13" x2="19.9" y2="19.5" width="0.3048" layer="16"/>
-<wire x1="19.9" y1="19.5" x2="19.9" y2="18.1" width="0.3048" layer="16"/>
-<wire x1="8.22" y1="57.07" x2="8.22" y2="55.18" width="0.4064" layer="16"/>
-<wire x1="8.22" y1="55.18" x2="12.5" y2="50.9" width="0.4064" layer="16"/>
-<wire x1="12.5" y1="50.9" x2="12.5" y2="20.1" width="0.4064" layer="16"/>
-<wire x1="12.5" y1="20.1" x2="15.04" y2="17.58" width="0.4064" layer="16"/>
-<wire x1="15.04" y1="17.58" x2="19.38" y2="17.58" width="0.3048" layer="16"/>
-<wire x1="19.38" y1="17.58" x2="19.9" y2="18.1" width="0.3048" layer="16"/>
-</signal>
-<signal name="N$6">
-<contactref element="X2" pad="9"/>
 <contactref element="IC1" pad="17"/>
-<wire x1="18.55" y1="27.74" x2="19.82" y2="26.47" width="0.3048" layer="16"/>
-<wire x1="19.82" y1="26.47" x2="19.82" y2="23.93" width="0.3048" layer="16"/>
-<wire x1="19.82" y1="23.93" x2="17.28" y2="21.39" width="0.3048" layer="16"/>
-<wire x1="15.3" y1="50.5" x2="15.3" y2="28.4" width="0.4064" layer="16"/>
-<wire x1="15.3" y1="50.5" x2="17.2" y2="52.4" width="0.4064" layer="16"/>
-<wire x1="17.2" y1="52.4" x2="17.2" y2="55.89" width="0.4064" layer="16"/>
-<wire x1="17.2" y1="55.89" x2="18.38" y2="57.07" width="0.4064" layer="16"/>
-<wire x1="18.55" y1="27.74" x2="15.96" y2="27.74" width="0.3048" layer="16"/>
-<wire x1="15.96" y1="27.74" x2="15.3" y2="28.4" width="0.3048" layer="16"/>
+<wire x1="17.28" y1="21.39" x2="18.45" y2="21.39" width="0.4064" layer="16"/>
+<wire x1="18.45" y1="21.39" x2="19.82" y2="20.02" width="0.4064" layer="16"/>
+<wire x1="19.82" y1="20.02" x2="19.82" y2="18.72" width="0.4064" layer="16"/>
+<wire x1="19.82" y1="18.72" x2="18.75" y2="17.65" width="0.4064" layer="16"/>
+<wire x1="18.75" y1="17.65" x2="18.74" y2="17.65" width="0.4064" layer="16"/>
+<wire x1="18.74" y1="17.65" x2="18.67" y2="17.58" width="0.4064" layer="16"/>
+<wire x1="18.67" y1="17.58" x2="14.51" y2="17.58" width="0.4064" layer="16"/>
+<wire x1="14.51" y1="17.58" x2="12.45" y2="19.64" width="0.4064" layer="16"/>
+<wire x1="12.45" y1="19.64" x2="12.45" y2="53.17" width="0.4064" layer="16"/>
+<wire x1="12.45" y1="53.17" x2="10.64" y2="54.98" width="0.4064" layer="16"/>
+<wire x1="10.64" y1="54.98" x2="9.23" y2="54.98" width="0.4064" layer="16"/>
+<wire x1="9.23" y1="54.98" x2="8.21" y2="56" width="0.4064" layer="16"/>
+<wire x1="8.21" y1="56" x2="8.21" y2="57.06" width="0.4064" layer="16"/>
+<wire x1="8.21" y1="57.06" x2="8.22" y2="57.07" width="0.4064" layer="16"/>
 </signal>
 <signal name="N$9">
@@
 <wire x1="18.08" y1="41.71" x2="20.6" y2="44.23" width="0.4064" layer="16"/>
 </signal>
+<signal name="N$27">
+<contactref element="IC1" pad="18"/>
+<contactref element="X2" pad="9"/>
+<wire x1="18.38" y1="57.07" x2="18.38" y2="53.14" width="0.4064" layer="16"/>
+<wire x1="18.38" y1="53.14" x2="15.34" y2="50.1" width="0.4064" layer="16"/>
+<wire x1="15.34" y1="50.1" x2="15.34" y2="28.44" width="0.4064" layer="16"/>
+<wire x1="15.34" y1="28.44" x2="16.07" y2="27.71" width="0.4064" layer="16"/>
+<wire x1="16.07" y1="27.71" x2="18.38" y2="27.71" width="0.4064" layer="16"/>
+<wire x1="18.38" y1="27.71" x2="19.72" y2="26.37" width="0.4064" layer="16"/>
+<wire x1="19.72" y1="26.37" x2="19.72" y2="24.74" width="0.4064" layer="16"/>
+<wire x1="19.72" y1="24.74" x2="18.93" y2="23.95" width="0.4064" layer="16"/>
+<wire x1="18.93" y1="23.95" x2="17.3" y2="23.95" width="0.4064" layer="16"/>
+<wire x1="17.3" y1="23.95" x2="17.28" y2="23.93" width="0.4064" layer="16"/>
+</signal>
 </signals>

Commit message: Add files via upload
Connections:
- net N$27: now also X2.1; no longer X2.9
- net N$3: now also X2.9; no longer X2.1
Routing:
- net N$27: track 39.5 -> 59.3 mm
- net N$3: track 53.1 -> 41.6 mm
Changed lines of the file:
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@@
 </polygon>
 <contactref element="JP4" pad="2"/>
-<wire x1="9.66" y1="31.55" x2="17.28" y2="34.09" width="0" layer="19" extent="1-1"/>
+<wire x1="17.28" y1="34.09" x2="9.66" y2="31.55" width="0" layer="19" extent="1-1"/>
 </signal>
 <signal name="N$5">
@@
 <wire x1="8.969" y1="13.01" x2="11.391" y2="13.01" width="0.4064" layer="16"/>
 <wire x1="11.391" y1="13.01" x2="11.431" y2="12.97" width="0.4064" layer="16"/>
-<wire x1="5.39" y1="10.68" x2="5.78" y2="10.68" width="0.4064" layer="16"/>
 <wire x1="5.78" y1="10.68" x2="7.5" y2="12.4" width="0.4064" layer="16"/>
 <wire x1="7.5" y1="12.4" x2="8.359" y2="12.4" width="0.4064" layer="16"/>
 <wire x1="8.359" y1="12.4" x2="8.969" y2="13.01" width="0.4064" layer="16"/>
+<wire x1="5.39" y1="10.68" x2="5.78" y2="10.68" width="0.4064" layer="16"/>
 </signal>
 <signal name="N$8">
@@
 <wire x1="9.45" y1="16.1" x2="9.66" y2="16.31" width="0.4064" layer="16"/>
 </signal>
-<signal name="N$3">
-<contactref element="X2" pad="1"/>
-<contactref element="IC1" pad="17"/>
-<wire x1="17.28" y1="21.39" x2="18.45" y2="21.39" width="0.4064" layer="16"/>
-<wire x1="18.45" y1="21.39" x2="19.82" y2="20.02" width="0.4064" layer="16"/>
-<wire x1="19.82" y1="20.02" x2="19.82" y2="18.72" width="0.4064" layer="16"/>
-<wire x1="19.82" y1="18.72" x2="18.75" y2="17.65" width="0.4064" layer="16"/>
-<wire x1="18.75" y1="17.65" x2="18.74" y2="17.65" width="0.4064" layer="16"/>
-<wire x1="18.74" y1="17.65" x2="18.67" y2="17.58" width="0.4064" layer="16"/>
-<wire x1="18.67" y1="17.58" x2="14.51" y2="17.58" width="0.4064" layer="16"/>
-<wire x1="14.51" y1="17.58" x2="12.45" y2="19.64" width="0.4064" layer="16"/>
-<wire x1="12.45" y1="19.64" x2="12.45" y2="53.17" width="0.4064" layer="16"/>
-<wire x1="12.45" y1="53.17" x2="10.64" y2="54.98" width="0.4064" layer="16"/>
-<wire x1="10.64" y1="54.98" x2="9.23" y2="54.98" width="0.4064" layer="16"/>
-<wire x1="9.23" y1="54.98" x2="8.21" y2="56" width="0.4064" layer="16"/>
-<wire x1="8.21" y1="56" x2="8.21" y2="57.06" width="0.4064" layer="16"/>
-<wire x1="8.21" y1="57.06" x2="8.22" y2="57.07" width="0.4064" layer="16"/>
-</signal>
 <signal name="N$9">
 </signal>
@@
 <signal name="N$27">
 <contactref element="IC1" pad="18"/>
+<contactref element="X2" pad="1"/>
+<wire x1="17.28" y1="23.93" x2="15.55" y2="23.93" width="0.4064" layer="16"/>
+<wire x1="15.55" y1="23.93" x2="14.95" y2="23.33" width="0.4064" layer="16"/>
+<wire x1="14.95" y1="23.33" x2="14.95" y2="20.97" width="0.4064" layer="16"/>
+<wire x1="14.95" y1="20.97" x2="15.81" y2="20.11" width="0.4064" layer="16"/>
+<wire x1="15.81" y1="20.11" x2="18.57" y2="20.11" width="0.4064" layer="16"/>
+<wire x1="18.57" y1="20.11" x2="19.4" y2="19.28" width="0.4064" layer="16"/>
+<wire x1="19.4" y1="19.28" x2="19.4" y2="18.34" width="0.4064" layer="16"/>
+<wire x1="19.4" y1="18.34" x2="18.64" y2="17.58" width="0.4064" layer="16"/>
+<wire x1="18.64" y1="17.58" x2="14.61" y2="17.58" width="0.4064" layer="16"/>
+<wire x1="14.61" y1="17.58" x2="12.48" y2="19.71" width="0.4064" layer="16"/>
+<wire x1="12.48" y1="19.71" x2="12.48" y2="19.76" width="0.4064" layer="16"/>
+<wire x1="12.48" y1="19.76" x2="12.45" y2="19.79" width="0.4064" layer="16"/>
+<wire x1="12.45" y1="19.79" x2="12.45" y2="53.97" width="0.3048" layer="16"/>
+<wire x1="12.45" y1="53.97" x2="11.33" y2="55.09" width="0.4064" layer="16"/>
+<wire x1="11.33" y1="55.09" x2="9.52" y2="55.09" width="0.4064" layer="16"/>
+<wire x1="9.52" y1="55.09" x2="8.25" y2="56.36" width="0.4064" layer="16"/>
+<wire x1="8.25" y1="56.36" x2="8.25" y2="57.04" width="0.4064" layer="16"/>
+<wire x1="8.25" y1="57.04" x2="8.22" y2="57.07" width="0.4064" layer="16"/>
+</signal>
+<signal name="N$3">
 <contactref element="X2" pad="9"/>
-<wire x1="18.38" y1="57.07" x2="18.38" y2="53.14" width="0.4064" layer="16"/>
-<wire x1="18.38" y1="53.14" x2="15.34" y2="50.1" width="0.4064" layer="16"/>
-<wire x1="15.34" y1="50.1" x2="15.34" y2="28.44" width="0.4064" layer="16"/>
-<wire x1="15.34" y1="28.44" x2="16.07" y2="27.71" width="0.4064" layer="16"/>
-<wire x1="16.07" y1="27.71" x2="18.38" y2="27.71" width="0.4064" layer="16"/>
-<wire x1="18.38" y1="27.71" x2="19.72" y2="26.37" width="0.4064" layer="16"/>
-<wire x1="19.72" y1="26.37" x2="19.72" y2="24.74" width="0.4064" layer="16"/>
-<wire x1="19.72" y1="24.74" x2="18.93" y2="23.95" width="0.4064" layer="16"/>
-<wire x1="18.93" y1="23.95" x2="17.3" y2="23.95" width="0.4064" layer="16"/>
-<wire x1="17.3" y1="23.95" x2="17.28" y2="23.93" width="0.4064" layer="16"/>
+<contactref element="IC1" pad="17"/>
+<wire x1="18.38" y1="57.07" x2="18.38" y2="53.48" width="0.4064" layer="16"/>
+<wire x1="18.38" y1="53.48" x2="15.51" y2="50.61" width="0.4064" layer="16"/>
+<wire x1="15.51" y1="50.61" x2="15.49" y2="50.61" width="0.4064" layer="16"/>
+<wire x1="15.49" y1="50.61" x2="15.27" y2="50.39" width="0.4064" layer="16"/>
+<wire x1="15.27" y1="50.39" x2="15.27" y2="28.36" width="0.3048" layer="16"/>
+<wire x1="15.27" y1="28.36" x2="15.85" y2="27.78" width="0.4064" layer="16"/>
+<wire x1="15.85" y1="27.78" x2="15.88" y2="27.78" width="0.4064" layer="16"/>
+<wire x1="15.88" y1="27.78" x2="15.92" y2="27.74" width="0.4064" layer="16"/>
+<wire x1="15.92" y1="27.74" x2="18.39" y2="27.74" width="0.4064" layer="16"/>
+<wire x1="18.39" y1="27.74" x2="19.47" y2="26.66" width="0.4064" layer="16"/>
+<wire x1="19.47" y1="26.66" x2="19.47" y2="22.71" width="0.4064" layer="16"/>
+<wire x1="19.47" y1="22.71" x2="18.17" y2="21.41" width="0.4064" layer="16"/>
+<wire x1="18.17" y1="21.41" x2="17.3" y2="21.41" width="0.4064" layer="16"/>
+<wire x1="17.3" y1="21.41" x2="17.28" y2="21.39" width="0.4064" layer="16"/>
 </signal>
 </signals>
