File: Programmer/USBasp_B.sch (EAGLE design)
At the start: 20 parts, among them IC1 ATMega8, Q1 12MHz

Commit message: Add files via upload
Connections:
- removed net N$6: IC1.PB3(MOSI/OC2), X2.9
- new net N$27: IC1.PB4(MISO), X2.9
- net N$3: now also IC1.PB3(MOSI/OC2); no longer IC1.PB4(MISO)
Changed lines of the file:
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@@
 <segment>
 <pinref part="X2" gate="G$1" pin="1"/>
-<wire x1="129.54" y1="116.84" x2="99.06" y2="116.84" width="0.1524" layer="91"/>
-<wire x1="99.06" y1="116.84" x2="96.52" y2="114.3" width="0.1524" layer="91"/>
-<pinref part="IC1" gate="G$1" pin="PB4(MISO)"/>
-<wire x1="96.52" y1="114.3" x2="68.58" y2="114.3" width="0.1524" layer="91"/>
-</segment>
-</net>
-<net name="N$6" class="0">
-<segment>
-<pinref part="X2" gate="G$1" pin="9"/>
-<wire x1="129.54" y1="106.68" x2="93.98" y2="106.68" width="0.1524" layer="91"/>
-<wire x1="93.98" y1="106.68" x2="83.82" y2="116.84" width="0.1524" layer="91"/>
+<wire x1="129.54" y1="116.84" x2="68.58" y2="116.84" width="0.1524" layer="91"/>
 <pinref part="IC1" gate="G$1" pin="PB3(MOSI/OC2)"/>
-<wire x1="83.82" y1="116.84" x2="68.58" y2="116.84" width="0.1524" layer="91"/>
 </segment>
 </net>
@@
 </segment>
 </net>
+<net name="N$27" class="0">
+<segment>
+<pinref part="IC1" gate="G$1" pin="PB4(MISO)"/>
+<wire x1="101.6" y1="114.3" x2="68.58" y2="114.3" width="0.1524" layer="91"/>
+<wire x1="101.6" y1="114.3" x2="101.6" y2="106.68" width="0.1524" layer="91"/>
+<pinref part="X2" gate="G$1" pin="9"/>
+<wire x1="101.6" y1="106.68" x2="129.54" y2="106.68" width="0.1524" layer="91"/>
+</segment>
+</net>

Commit message: Add files via upload
Connections:
- net N$27: now also X2.1; no longer X2.9
- net N$3: now also X2.9; no longer X2.1
Changed lines of the file:
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@@
-</segment>
-</net>
-<net name="N$3" class="0">
-<segment>
-<pinref part="X2" gate="G$1" pin="1"/>
-<wire x1="129.54" y1="116.84" x2="68.58" y2="116.84" width="0.1524" layer="91"/>
-<pinref part="IC1" gate="G$1" pin="PB3(MOSI/OC2)"/>
 </segment>
 </net>
@@
 <segment>
 <pinref part="IC1" gate="G$1" pin="PB4(MISO)"/>
-<wire x1="101.6" y1="114.3" x2="68.58" y2="114.3" width="0.1524" layer="91"/>
-<wire x1="101.6" y1="114.3" x2="101.6" y2="106.68" width="0.1524" layer="91"/>
-<pinref part="X2" gate="G$1" pin="9"/>
-<wire x1="101.6" y1="106.68" x2="129.54" y2="106.68" width="0.1524" layer="91"/>
+<wire x1="124.46" y1="114.3" x2="68.58" y2="114.3" width="0.1524" layer="91"/>
+<wire x1="124.46" y1="114.3" x2="124.46" y2="116.84" width="0.1524" layer="91"/>
+<pinref part="X2" gate="G$1" pin="1"/>
+<wire x1="124.46" y1="116.84" x2="129.54" y2="116.84" width="0.1524" layer="91"/>
 </segment>
 </net>
+<net name="N$3" class="0">
+<segment>
+<pinref part="X2" gate="G$1" pin="9"/>
+<wire x1="99.06" y1="106.68" x2="129.54" y2="106.68" width="0.1524" layer="91"/>
+<wire x1="99.06" y1="106.68" x2="99.06" y2="116.84" width="0.1524" layer="91"/>
+<pinref part="IC1" gate="G$1" pin="PB3(MOSI/OC2)"/>
+<wire x1="99.06" y1="116.84" x2="68.58" y2="116.84" width="0.1524" layer="91"/>
+</segment>
+</net>

Commit message: Add files via upload
Other:
- note removed: "Prashant kumar"
Changed lines of the file:
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@@
 <sheet>
 <plain>
-<text x="119.38" y="48.26" size="2.54" layer="94">Prashant kumar</text>
 </plain>
 <instances>
